Commit message: changed according to Steve's package and tested. a big urdf file was added

File: gazebo/gazebo.urdf.xacro (robot description, xacro)
@@ -4,11 +4,10 @@
 		<plugin name="gazebo_ros_controller_manager" filename="libgazebo_ros_control.so">
 			<robotNamespace>/hyq</robotNamespace>
-			<robotSimType>dls_gazebo_interface/DLSHWSim</robotSimType>
-			<controlPeriod>0.004</controlPeriod>
+			<controlPeriod>0.001</controlPeriod>
 		</plugin>
 		<plugin filename="libgazebo_ros_p3d.so" name="gazebo_ros_p3d">
 			<robotNamespace>/hyq</robotNamespace>
 		 	<bodyName>trunk</bodyName>
-			<topicName>ground_truth</topicName>
+			<topicName>ground_truth_odom</topicName>
 			<frameName>world</frameName>
 			<xyzOffsets>0 0 0</xyzOffsets>
@@ -16,5 +15,5 @@
 			<gaussianNoise>0</gaussianNoise>
 			<alwaysOn>true</alwaysOn>
-			<updateRate>250.0</updateRate>
+			<updateRate>200.0</updateRate>
 		</plugin>
 	</gazebo>

File: robots/hyq.urdf.xacro (robot description, xacro)
@@ -3,5 +3,4 @@
 	<!-- The following included files set up definitions of parts of the robot body -->
 	<xacro:include filename="$(find hyq_description)/urdfs/common.xacro"/>
-	<xacro:include filename="$(find sensors_description)/urdfs/common.xacro"/>
 	<!-- HyQ trunk -->
 	<xacro:include filename="$(find hyq_description)/urdfs/trunk/trunk.urdf.xacro"/>
@@ -9,14 +8,11 @@
 	<xacro:include filename="$(find hyq_description)/urdfs/leg/leg.urdf.xacro"/>
 	<!-- HyQ sensors -->
-	<xacro:include filename="$(find sensors_description)/urdfs/sensors/microstrain_3dmgx425_imu.urdf.xacro"/>
-	<xacro:include filename="$(find sensors_description)/urdfs/sensors/asus_xtion.urdf.xacro"/>
-	<!-- Velodyne disabled because it takes too long to load-up -->
-	<!-- <xacro:include filename="$(find sensors_description)/urdfs/sensors/velodyne.urdf.xacro"/> -->
-	<xacro:include filename="$(find sensors_description)/urdfs/sensors/kinect.urdf.xacro"/>
-	<xacro:include filename="$(find sensors_description)/urdfs/sensors/ptu_d46.urdf.xacro"/>
-	<xacro:include filename="$(find sensors_description)/urdfs/sensors/bumblebee.urdf.xacro"/>
-	<xacro:include filename="$(find sensors_description)/urdfs/sensors/vislab_3dve.urdf.xacro"/>
-	<xacro:include filename="$(find sensors_description)/urdfs/sensors/hokuyo_laser.urdf.xacro"/>
-	<xacro:include filename="$(find sensors_description)/urdfs/sensors/multisense_sl.urdf.xacro"/>
+	<xacro:include filename="$(find hyq_description)/urdfs/sensors/microstrain_3dmgx325_imu.urdf.xacro"/>
+	<xacro:include filename="$(find hyq_description)/urdfs/sensors/asus_xtion.urdf.xacro"/>
+	<xacro:include filename="$(find hyq_description)/urdfs/sensors/velodyne.urdf.xacro"/>
+	<xacro:include filename="$(find hyq_description)/urdfs/sensors/kinect.urdf.xacro"/>
+	<xacro:include filename="$(find hyq_description)/urdfs/sensors/ptu_d46.urdf.xacro"/>
+	<xacro:include filename="$(find hyq_description)/urdfs/sensors/bumblebee.urdf.xacro"/>
+	<xacro:include filename="$(find hyq_description)/urdfs/sensors/vislab_3dve.urdf.xacro"/>
 	<!-- generic simulator_gazebo plugins for starting mechanism control, ros time -->
 	<xacro:include filename="$(find hyq_description)/gazebo/gazebo.urdf.xacro"/>
@@ -71,39 +67,52 @@
 	</xacro:hyq_leg>
 	<!-- IMU trunk -->
-	<xacro:microstrain_3dmgx425_imu
+	<xacro:microstrain_3dmgx325_imu
 		parent="trunk"
-		imu_name="imu"
+		imu_name="3dmgx325_trunk_imu"
 		imu_topic="trunk_imu/data"
-		update_rate="250"
-		rate_mean="0"
-		rate_stddev="2e-4"
-		rate_bias_mean="0.00087"
-		rate_bias_stddev="0.0000008"
-		accel_mean="0"
-		accel_stddev="1.7e-2"
-		accel_bias_mean="0.002"
-		accel_bias_stddev="0.001">
-		<origin xyz="0.290 0.000 0.0999214" rpy="0 ${-PI} 0"/>
-	</xacro:microstrain_3dmgx425_imu>
-	<!-- Hokuyo -->
-	<xacro:hokuyo_laser
-		name="laser"
-		parent="trunk"
-		ros_topic="scan"
-		update_rate="10"
-		min_angle="-5"
-		max_angle="5"
-		range="4.0">
-	<origin xyz="0.475 0.0 -0.08823" rpy="3.14 0.0 0"/>
-	</xacro:hokuyo_laser>
-    <xacro:multisense_sl parent="trunk" prefix="hyq">
-            <!-- <origin xyz="0.741737 0.0191395 0.143229" rpy="-0.0241345 0.446222 -0.0347202"/> -->
-            <origin xyz="0.741737 0.0 0.143229" rpy="-0.0241345 0.446222 -0.0347202"/>
-    </xacro:multisense_sl>
+		update_rate="100.0"
+		stdev="0.00017">
+		<origin xyz="0.3 0 0.095" rpy="0 ${-PI} 0"/>
+	</xacro:microstrain_3dmgx325_imu>
+	<!-- Velodyne -->
+	<xacro:velodyne
+		name="trunk_mount"
+		parent="trunk">
+		<origin xyz="0.39 0 0.269" rpy="0 0 0"/>
+	</xacro:velodyne>
+	<!-- PTU unit -->
+	<xacro:ptu_d46
+		name="ptu"
+		parent="trunk">
+		<origin xyz="0.657353 0.015447 0.119533" rpy="-0.013127 0.569257 -0.007748"/>
+<!--		<origin xyz="0.667353 -0.010101 0.160544" rpy="0.043239 0.569257 0.041771"/>-->
+	</xacro:ptu_d46>
 	<!-- Asus Xtion Pro -->
 	<!--<origin xyz="0 0.005 0.036" rpy="0 0 0"/> with Bumblebee setup -->
 	<!--<origin xyz="0 0 0.04397" rpy="0 0 0"/> with Vislab setup -->
-	<xacro:asus_xtion_camera name="asus" parent="trunk">
-		<origin xyz="0.66489 0.0016545 0.0380496" rpy="0.00740313 0.479116 0.0244919"/>
+	<xacro:asus_xtion_camera
+		name="head_mount"
+		parent="ptu_mount_link">
+		<origin xyz="0 0.005 0.036" rpy="0 0 0"/>
 	</xacro:asus_xtion_camera>
+	<!-- Kinect --> <!-- is no more used, but we keep it for compatibilty -->
+	<!--xacro:kinect_camera
+		name="head_mount"
+		parent="trunk">
+		<origin xyz="0.63 0 0.095" rpy="0 0 0"/>
+	</xacro:kinect_camera-->
+	<!-- Bumblebee -->
+	<xacro:bumblebee_97
+		parent_link="ptu_mount_link"
+		xyz="0 0 0.018"
+		rpy="0 0 0"
+		ns="bumblebee"
+		frame_prefix="bumblebee_"
+		high_res="false"/>
+<!--	<xacro:vislab_3dve_72
+		name="vislab_3dve"
+		parent="ptu_mount_link"
+		xyz="0 0 0.025"
+		rpy="0 0 0"
+		high_res="false"/>-->
 </robot>

File: urdfs/common.xacro (robot description, xacro)
@@ -5,19 +5,18 @@
 	<property name="d_lr" value="0.414"/>
 	<property name="d_fh" value="0.747"/>
-	<property name="d_p0p1" value="0.08"/>
+	<property name="d_tbb" value="0.082"/>
 	<property name="d_p1p2" value="0.35"/>
-	<property name="d_p2p3" value="0.341"/>
 	<!-- Inertial values -->
 	<!-- Trunk with hydraulic system -->
-	<property name="xcom_trunk" value="0.02255"/>
-	<property name="ycom_trunk" value="-0.0035"/>
-	<property name="zcom_trunk" value="0.018"/>
-	<property name="m_trunk" value="63.8"/>
-	<property name="ixx_trunk" value="1.5725937"/>
-	<property name="iyy_trunk" value="8.5015928"/>
-	<property name="izz_trunk" value="9.1954911"/>
-	<property name="ixy_trunk" value="0.028375"/>
-	<property name="ixz_trunk" value="-0.203139"/>
-	<property name="iyz_trunk" value="-0.004462"/>
+	<property name="xcom_trunk" value="-0.02758"/>
+	<property name="ycom_trunk" value="-0.000023319"/>
+	<property name="zcom_trunk" value="0.03103"/>
+	<property name="m_trunk" value="50.24"/>
+	<property name="ixx_trunk" value="0.97322"/>
+	<property name="iyy_trunk" value="5.0487"/>
+	<property name="izz_trunk" value="5.283"/>
+	<property name="ixy_trunk" value="-0.0067362"/>
+	<property name="ixz_trunk" value="0.1681"/>
+	<property name="iyz_trunk" value="-0.0060307"/>
 	<!-- Hip assembly -->
 	<property name="xcom_hipassembly" value="0.04263"/>
@@ -25,10 +24,10 @@
 	<property name="zcom_hipassembly" value="0.16931"/>
 	<property name="m_hipassembly" value="2.93"/>
-	<property name="ixx_hipassembly" value="0.05071"/>
-	<property name="iyy_hipassembly" value="0.05486"/>
-	<property name="izz_hipassembly" value="0.00571"/>
-	<property name="ixy_hipassembly" value="-0.00004"/>
-	<property name="ixz_hipassembly" value="-0.00159"/>
-	<property name="iyz_hipassembly" value="-0.00005"/>
+	<property name="ixx_hipassembly" value="0.134705"/>
+	<property name="iyy_hipassembly" value="0.144171"/>
+	<property name="izz_hipassembly" value="0.011033"/>
+	<property name="ixy_hipassembly" value="0.000036"/>
+	<property name="ixz_hipassembly" value="0.022734"/>
+	<property name="iyz_hipassembly" value="0.000051"/>
 	<!-- Upper leg -->
 	<property name="xcom_upperleg" value="0.15074"/>
@@ -36,20 +35,59 @@
 	<property name="zcom_upperleg" value="0.0"/>
 	<property name="m_upperleg" value="2.638"/>
-	<property name="ixx_upperleg" value="0.00368"/>
-	<property name="iyy_upperleg" value="0.02719"/>
-	<property name="izz_upperleg" value="0.02811"/>
-	<property name="ixy_upperleg" value="-0.00302"/>
-	<property name="ixz_upperleg" value="0.0001"/>
-	<property name="iyz_upperleg" value="0.00002"/>
+	<property name="ixx_upperleg" value="0.005495"/>
+	<property name="iyy_upperleg" value="0.087136"/>
+	<property name="izz_upperleg" value="0.089871"/>
+	<property name="ixy_upperleg" value="-0.007418"/>
+	<property name="ixz_upperleg" value="-0.000102"/>
+	<property name="iyz_upperleg" value="-0.000021"/>
 	<!-- Lower leg -->
 	<property name="xcom_lowerleg" value="0.1254"/>
-	<property name="ycom_lowerleg" value="0.00004"/>
+	<property name="ycom_lowerleg" value="0.00005"/>
 	<property name="zcom_lowerleg" value="-0.0001"/>
 	<property name="m_lowerleg" value="0.881"/>
-	<property name="ixx_lowerleg" value="0.00047"/>
-	<property name="iyy_lowerleg" value="0.01256"/>
-	<property name="izz_lowerleg" value="0.01233"/>
-	<property name="ixy_lowerleg" value="0.00006"/>
-	<property name="ixz_lowerleg" value="-0.00001"/>
-	<property name="iyz_lowerleg" value="-0.0"/>
+	<property name="ixx_lowerleg" value="0.000468"/>
+	<property name="iyy_lowerleg" value="0.026409"/>
+	<property name="izz_lowerleg" value="0.026181"/>
+	<property name="ixy_lowerleg" value="0.0"/>
+	<property name="ixz_lowerleg" value="0.0"/>
+	<property name="iyz_lowerleg" value="0.0"/>
+	<!-- PTU unit -->
+	<property name="pan_velocity" value="1.0" />
+	<property name="pan_range" value="2.775" />
+	<property name="tilt_velocity" value="1.0" />
+	<property name="tilt_up_range" value="0.52" />
+	<property name="tilt_down_range" value="0.82" />
+	<property name="joint_effort" value="30" />
+	<!-- Asus Xtion Camera Location (Nominally 0) -->
+	<property name="asus_xtion_x" value="0.009"/>
+	<property name="asus_xtion_depth_y" value="0.045"/>
+	<property name="asus_xtion_rgb_y" value="0.01875"/>
+	<property name="asus_xtion_z" value="0.035"/>
+	<property name="asus_xtion_roll" value="${-PI/2}"/>
+	<property name="asus_xtion_pitch" value="0.0"/>
+	<property name="asus_xtion_yaw" value="${-PI/2}"/>
+	<!-- Kinect Camera Location (Nominally 0) -->
+	<property name="kinect_x" value="0.025"/>
+	<property name="kinect_ir_y" value="0.01"/>
+	<property name="kinect_rgb_y" value="0.015"/>
+	<property name="kinect_z" value="0.052"/>
+	<property name="kinect_roll" value="${-PI/2}"/>
+	<property name="kinect_pitch" value="0.0"/>
+	<property name="kinect_yaw" value="${-PI/2}"/>
+	<!-- Bumblebee mass and lengths for computing inertia tensor -->
+	<property name="b2mass" value="0.342"/>
+	<property name="b2lx" value="0.157"/>
+	<property name="b2ly" value="0.036"/>
+	<property name="b2lz" value="0.0474"/>
+	<!-- Velodyne Lidar Location (Nominally 0) -->
+	<property name="velodyne_x" value="0.0"/>
+	<property name="velodyne_y" value="0.0"/>
+	<property name="velodyne_z" value="0.09"/>
+	<!-- HighDef Camera Location (Nominally 0) -->
+	<property name="cal_high_def_x" value="0.0" />
+	<property name="cal_high_def_y" value="0.0" />
+	<property name="cal_high_def_z" value="0.0" />
+	<property name="cal_high_def_roll" value="0.0" />
+	<property name="cal_high_def_pitch" value="0.0" />
+	<property name="cal_high_def_yaw" value="0.0" />
 </robot>

File: urdfs/leg/leg.gazebo.xacro (robot description, xacro)
@@ -2,13 +2,4 @@
 <robot xmlns:xacro="http://www.ros.org/wiki/xacro">
 	<xacro:macro name="leg_gazebo" params="name">
-		<gazebo reference="${name}_upperleg">
-			<kp>1000000.0</kp>
-			<kd>100.0</kd>
-			<mu1>1.5</mu1>
-			<mu2>1.5</mu2>
-			<fdir1>1 0 0</fdir1>
-			<maxVel>1.0</maxVel>
-			<minDepth>0.00</minDepth>
-		</gazebo>
 		<gazebo reference="${name}_lowerleg">
 			<kp>1000000.0</kp>
@@ -20,15 +11,4 @@
 			<minDepth>0.00</minDepth>
 		</gazebo>
-		<gazebo reference="${name}_foot">
-			<!-- contact sensor -->
-			<sensor type="contact" name="${name}_foot_contact_sensor">
-				<update_rate>1000.0</update_rate>
-				<always_on>1</always_on>
-				<contact>
-					<collision>${name}_foot_collision</collision>
-					<topic>/${name}_foot_contact</topic>
-				</contact>
-			</sensor>
-		</gazebo>
 	</xacro:macro>
 </robot>

File: urdfs/leg/leg.transmission.xacro (robot description, xacro)
@@ -14,5 +14,5 @@
 		</transmission>
     	<!-- Upper leg -->
-		<transmission name="${name}_hfe_trans">
+		<transmission name="${name}_hfe_upper_trans">
 			<type>transmission_interface/SimpleTransmission</type>
 			<joint name="${name}_hfe_joint">

File: urdfs/leg/leg.urdf.xacro (robot description, xacro)
@@ -14,12 +14,12 @@
 			<child  link="${name}_hipassembly"/>
 			<axis xyz="0 0 1"/>
-			<limit effort="150.0" velocity="12.0" lower="${-7*PI/18}" upper="${5*PI/36}"/>
+			<limit effort="150.0" velocity="12.0" lower="${-7*PI/18}" upper="${PI/6}"/>
 			<dynamics damping="0.1" friction="0" />
 			<safety_controller k_position="100" k_velocity="100"
-							   soft_lower_limit="${-7*PI/18}" soft_upper_limit="${5*PI/36}" />
+							   soft_lower_limit="${-7*PI/18}" soft_upper_limit="${PI/6}" />
 		</joint>
 		<!-- Upper leg joint -->
 		<joint name="${name}_hfe_joint" type="revolute">
-			<origin xyz="${d_p0p1} 0 0" rpy="${reflect_upper*PI/2} 0 0"/>
+			<origin xyz="${d_tbb} 0 0" rpy="${reflect_upper*PI/2} 0 0"/>
 			<parent link="${name}_hipassembly"/>
 			<child  link="${name}_upperleg"/>
@@ -49,5 +49,5 @@
 		</joint>
 		<joint name="${name}_foot_joint" type="fixed">
-			<origin xyz="${d_p2p3} 0 0" rpy="${PI/2} 0 ${-PI/2}"/>
+			<origin xyz="0.35 0 0" rpy="${PI/2} 0 ${-PI/2}"/>
 			<parent link="${name}_lowerleg"/>
 			<child  link="${name}_foot"/>
@@ -62,5 +62,5 @@
 				<mass value="${m_hipassembly}"/>
 				<inertia ixx="${ixx_hipassembly}" iyy="${iyy_hipassembly}" izz="${izz_hipassembly}"
-						 ixy="${reflect_hip*ixy_hipassembly}" ixz="${reflect_hip*ixz_hipassembly}" iyz="${iyz_hipassembly}"/>
+						 ixy="${reflect_hip*reflect_front*ixy_hipassembly}" ixz="${reflect_hip*reflect_front*ixz_hipassembly}" iyz="${iyz_hipassembly}"/>
 			</inertial>
 			<visual>
@@ -80,5 +80,5 @@
 		<link name="${name}_upperleg">
 			<inertial>
-				<origin xyz="${xcom_upperleg} ${-reflect_front*ycom_upperleg} ${zcom_upperleg}"/>
+				<origin xyz="${xcom_upperleg} ${reflect_upper*ycom_upperleg} ${zcom_upperleg}"/>
 				<mass value="${m_upperleg}"/>
 				<inertia ixx="${ixx_upperleg}" iyy="${iyy_upperleg}" izz="${izz_upperleg}"
@@ -101,8 +101,8 @@
 		<link name="${name}_lowerleg">
 			<inertial>
-				<origin xyz="${xcom_lowerleg} ${reflect_front*ycom_lowerleg} ${reflect_front*zcom_lowerleg}"/>
+				<origin xyz="${xcom_lowerleg} ${ycom_lowerleg} ${zcom_lowerleg}"/>
 				<mass value="${m_lowerleg}"/>
 				<inertia ixx="${ixx_lowerleg}" iyy="${iyy_lowerleg}" izz="${izz_lowerleg}"
-						 ixy="${reflect_front*ixy_lowerleg}" ixz="${reflect_front*ixz_lowerleg}" iyz="${iyz_lowerleg}"/>
+						 ixy="${ixy_lowerleg}" ixz="${ixz_lowerleg}" iyz="${iyz_lowerleg}"/>
 			</inertial>
 			<visual>
@@ -122,7 +122,13 @@
 			<inertial>
 				<origin xyz="0 0 0"/>
-				<mass value="0.0"/>
+				<mass value="0.01"/>
 				<inertia ixx="0.0" iyy="0.0" izz="0.0" ixy="0.0" ixz="0.0" iyz="0.0"/>
 			</inertial>
+			<!--<visual>
+				<origin xyz="0.0 0.0 0.0" rpy="0.0 0.0 0.0"/>
+				<geometry>
+					<sphere radius="0.021"/>
+				</geometry>
+			</visual>-->
 			<collision>
 				<origin xyz="0 0 0" rpy="0 0 0"/>
